File: kicad/sentry-keyboard-v1.kicad_sch (KiCad schematic)
At the start: 269 parts, among them J2 Conn_01x04, J4 AVR-ISP-6, SW1 Reset, SW2 RotaryEncoder_Switch, U1 ATmega32U4-AU, Y1 16Mhz

Commit message: Update pins for encoder
I had the encoder and a switch on the same row/col
Connections:
- net Col12: no longer SW2.S1
- net Col13: now also SW2.S1
Other:
- note added: "The encoder switch is here"
Changed lines of the file:
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@@
 		)
 	)
+	(text "The encoder switch is here"
+		(exclude_from_sim no)
+		(at 388.62 98.552 0)
+		(effects
+			(font
+				(size 1.27 1.27)
+			)
+		)
+	)
 	(text "Key Matrix"
 		(exclude_from_sim no)
@@
 		)
 	)
-	(global_label "Col12"
+	(global_label "Col13"
 		(shape input)
 		(at 207.01 106.68 0)
