File: kicad/sentry-keyboard-v1.kicad_sch (KiCad schematic)
At the start: 269 parts, among them J2 Conn_01x04, J4 AVR-ISP-6, SW1 Reset, SW2 RotaryEncoder_Switch, U1 ATmega32U4-AU, Y1 16Mhz

Commit message: Update pins and fix routing
Connections:
- net Col12: now also U1.1 (PE6); no longer U1.38 (PF5)
- no-connect marks 4 -> 3
Changed lines of the file:
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@@
 	)
 	(no_connect
-		(at 96.52 105.41)
-	)
-	(no_connect
 		(at 274.32 374.65)
 	)
@@
 	(global_label "Col12"
 		(shape input)
-		(at 96.52 118.11 0)
+		(at 96.52 105.41 0)
 		(fields_autoplaced yes)
 		(effects
@@
 		)
 		(property "Intersheetrefs" "${INTERSHEET_REFS}"
-			(at 105.0084 118.11 0)
+			(at 105.0084 105.41 0)
 			(effects
 				(font

Commit message: Simplify encoder wiring
I built a prototype on a breadboard and the resistors and caps are not
required.
Parts:
- removed C8, C9: 100nF, Capacitor_SMD:C_0805_2012Metric, symbol Device:C
- removed R10, R9: 10k, Resistor_SMD:R_0805_2012Metric, symbol Device:R
Connections:
- no-connect marks 3 -> 4

Commit message: Flipped pins on USB connection
I had measured the pins on the daughter card, but the pins are reversed
on the mainboard.
Connections:
- net D+: now also R6.2; no longer R7.1
- net D-: now also R7.1; no longer R6.2
- net GND: now also J2.4 (Pin_4); no longer J2.1 (Pin_1)
- net VCC: now also J2.1 (Pin_1); no longer J2.4 (Pin_4)
Other:
- moved on the sheet: FU2, R6, R7
Changed lines of the file:
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@@
 	)
 	(junction
+		(at 158.75 50.8)
+		(diameter 0)
+		(color 0 0 0 0)
+	)
+	(junction
 		(at 342.9 87.63)
 		(diameter 0)
@@
 	)
 	(junction
-		(at 154.94 30.48)
-		(diameter 0)
-		(color 0 0 0 0)
-	)
-	(junction
 		(at 340.36 54.61)
 		(diameter 0)
@@
 	(wire
 		(pts
-			(xy 161.29 40.64) (xy 161.29 35.56)
+			(xy 161.29 36.83) (xy 161.29 35.56)
 		)
 		(stroke
@@
 	(wire
 		(pts
-			(xy 153.67 30.48) (xy 154.94 30.48)
-		)
-		(stroke
-			(width 0)
-			(type default)
-		)
-	)
-	(wire
-		(pts
 			(xy 181.61 250.19) (xy 181.61 255.27)
 		)
@@
 	(wire
 		(pts
-			(xy 168.91 36.83) (xy 171.45 36.83)
+			(xy 168.91 33.02) (xy 171.45 33.02)
 		)
 		(stroke
@@
 	(wire
 		(pts
-			(xy 154.94 30.48) (xy 160.02 30.48)
+			(xy 158.75 50.8) (xy 163.83 50.8)
 		)
 		(stroke
@@
 	(wire
 		(pts
-			(xy 165.1 30.48) (xy 172.72 30.48)
+			(xy 168.91 50.8) (xy 176.53 50.8)
 		)
 		(stroke
@@
 	(wire
 		(pts
-			(xy 163.83 36.83) (xy 162.56 36.83)
-		)
-		(stroke
-			(width 0)
-			(type default)
-		)
-	)
-	(wire
-		(pts
 			(xy 302.26 107.95) (xy 312.42 107.95)
 		)
@@
 	(wire
 		(pts
-			(xy 154.94 27.94) (xy 154.94 30.48)
+			(xy 158.75 48.26) (xy 158.75 50.8)
 		)
 		(stroke
@@
 	(wire
 		(pts
-			(xy 162.56 33.02) (xy 153.67 33.02)
+			(xy 153.67 33.02) (xy 163.83 33.02)
 		)
 		(stroke
@@
 	(wire
 		(pts
-			(xy 168.91 40.64) (xy 171.45 40.64)
+			(xy 168.91 36.83) (xy 171.45 36.83)
 		)
 		(stroke
@@
 	(wire
 		(pts
+			(xy 153.67 50.8) (xy 158.75 50.8)
+		)
+		(stroke
+			(width 0)
+			(type default)
+		)
+	)
+	(wire
+		(pts
 			(xy 139.7 241.3) (xy 160.02 241.3)
 		)
@@
 	(wire
 		(pts
-			(xy 160.02 38.1) (xy 160.02 45.72)
+			(xy 153.67 30.48) (xy 162.56 30.48)
 		)
 		(stroke
@@
 	(wire
 		(pts
-			(xy 160.02 38.1) (xy 153.67 38.1)
-		)
-		(stroke
-			(width 0)
-			(type default)
-		)
-	)
-	(wire
-		(pts
-			(xy 162.56 36.83) (xy 162.56 33.02)
-		)
-		(stroke
-			(width 0)
-			(type default)
-		)
-	)
-	(wire
-		(pts
 			(xy 203.2 387.35) (xy 224.79 387.35)
 		)
@@
 	(wire
 		(pts
+			(xy 153.67 38.1) (xy 153.67 50.8)
+		)
+		(stroke
+			(width 0)
+			(type default)
+		)
+	)
+	(wire
+		(pts
 			(xy 364.49 59.69) (xy 367.03 59.69)
 		)
@@
 	(wire
 		(pts
-			(xy 163.83 40.64) (xy 161.29 40.64)
+			(xy 163.83 36.83) (xy 161.29 36.83)
 		)
 		(stroke
@@
 		)
 	)
-	(global_label "D+"
+	(global_label "D-"
 		(shape input)
-		(at 171.45 40.64 0)
+		(at 171.45 36.83 0)
 		(effects
 			(font
@@
 		)
 		(property "Intersheetrefs" "${INTERSHEET_REFS}"
-			(at 171.45 40.64 0)
+			(at 171.45 36.83 0)
 			(effects
 				(font
@@
 		)
 	)
-	(global_label "D-"
+	(global_label "D+"
 		(shape input)
-		(at 171.45 36.83 0)
+		(at 171.45 33.02 0)
 		(effects
 			(font
@@
 		)
 		(property "Intersheetrefs" "${INTERSHEET_REFS}"
-			(at 171.45 36.83 0)
+			(at 171.45 33.02 0)
 			(effects
 				(font
@@
 	(symbol
 		(lib_id "Device:R_Small")
-		(at 166.37 40.64 270)
+		(at 166.37 36.83 270)
 		(unit 1)
 		(exclude_from_sim no)
@@
 		(dnp no)
 		(property "Reference" "R7"
-			(at 166.37 45.6184 90)
+			(at 166.37 41.8084 90)
 			(effects
 				(font
@@
 		)
 		(property "Value" "22"
-			(at 166.37 43.307 90)
+			(at 166.37 39.497 90)
 			(effects
 				(font
@@
 		)
 		(property "Footprint" "Resistor_SMD:R_0805_2012Metric"
-			(at 166.37 40.64 0)
+			(at 166.37 36.83 0)
 			(effects
 				(font
@@
 		)
 		(property "Datasheet" "~"
-			(at 166.37 40.64 0)
+			(at 166.37 36.83 0)
 			(effects
 				(font
@@
 		)
 		(property "Description" ""
-			(at 166.37 40.64 0)
+			(at 166.37 36.83 0)
 			(effects
 				(font
@@
 	(symbol
 		(lib_id "power:VCC")
-		(at 154.94 27.94 0)
+		(at 158.75 48.26 0)
 		(unit 1)
 		(exclude_from_sim no)
@@
 		(dnp no)
 		(property "Reference" "#PWR018"
-			(at 154.94 31.75 0)
+			(at 158.75 52.07 0)
 			(effects
 				(font
@@
 		)
 		(property "Value" "VCC"
-			(at 154.94 24.13 0)
+			(at 158.75 44.45 0)
 			(effects
 				(font
@@
 		)
 		(property "Footprint" ""
-			(at 154.94 27.94 0)
+			(at 158.75 48.26 0)
 			(effects
 				(font
@@
 		)
 		(property "Datasheet" ""
-			(at 154.94 27.94 0)
+			(at 158.75 48.26 0)
 			(effects
 				(font
@@
 		)
 		(property "Description" ""
-			(at 154.94 27.94 0)
+			(at 158.75 48.26 0)
 			(effects
 				(font
@@
 	(symbol
 		(lib_id "Device:Polyfuse_Small")
-		(at 162.56 30.48 270)
+		(at 166.37 50.8 270)
 		(unit 1)
 		(exclude_from_sim no)
@@
 		(dnp no)
 		(property "Reference" "FU2"
-			(at 162.56 25.273 90)
+			(at 166.37 45.593 90)
 			(effects
 				(font
@@
 		)
 		(property "Value" "500mA"
-			(at 162.56 27.5844 90)
+			(at 166.37 47.9044 90)
 			(effects
 				(font
@@
 		)
 		(property "Footprint" "Fuse:Fuse_1206_3216Metric_Pad1.42x1.75mm_HandSolder"
-			(at 157.48 31.75 0)
+			(at 161.29 52.07 0)
 			(effects
 				(font
@@
 		)
 		(property "Datasheet" "~"
-			(at 162.56 30.48 0)
+			(at 166.37 50.8 0)
 			(effects
 				(font
@@
 		)
 		(property "Description" ""
-			(at 162.56 30.48 0)
+			(at 166.37 50.8 0)
 			(effects
 				(font
@@
 	(symbol
 		(lib_id "power:GND")
-		(at 160.02 45.72 0)
+		(at 162.56 30.48 180)
 		(unit 1)
 		(exclude_from_sim no)
@@
 		(dnp no)
 		(property "Reference" "#PWR020"
-			(at 160.02 52.07 0)
+			(at 162.56 24.13 0)
 			(effects
 				(font
@@
 		)
 		(property "Value" "GND"
-			(at 160.147 50.1142 0)
+			(at 162.433 26.0858 0)
 			(effects
 				(font
@@
 		)
 		(property "Footprint" ""
-			(at 160.02 45.72 0)
+			(at 162.56 30.48 0)
 			(effects
 				(font
@@
 		)
 		(property "Datasheet" ""
-			(at 160.02 45.72 0)
+			(at 162.56 30.48 0)
 			(effects
 				(font
@@
 		)
 		(property "Description" ""
-			(at 160.02 45.72 0)
+			(at 162.56 30.48 0)
 			(effects
 				(font
@@
 	(symbol
 		(lib_id "Device:R_Small")
-		(at 166.37 36.83 90)
+		(at 166.37 33.02 90)
 		(unit 1)
 		(exclude_from_sim no)
@@
 		(dnp no)
 		(property "Reference" "R6"
-			(at 166.37 31.8516 90)
+			(at 166.37 28.0416 90)
 			(effects
 				(font
@@
 		)
 		(property "Value" "22"
-			(at 166.37 34.163 90)
+			(at 166.37 30.353 90)
 			(effects
 				(font
@@
 		)
 		(property "Footprint" "Resistor_SMD:R_0805_2012Metric"
-			(at 166.37 36.83 0)
+			(at 166.37 33.02 0)
 			(effects
 				(font
@@
 		)
 		(property "Datasheet" "~"
-			(at 166.37 36.83 0)
+			(at 166.37 33.02 0)
 			(effects
 				(font
@@
 		)
 		(property "Description" ""
-			(at 166.37 36.83 0)
+			(at 166.37 33.02 0)
 			(effects
 				(font
@@
 	(symbol
 		(lib_id "power:+5V")
-		(at 172.72 30.48 0)
+		(at 176.53 50.8 0)
 		(unit 1)
 		(exclude_from_sim no)
@@
 		(dnp no)
 		(property "Reference" "#PWR019"
-			(at 172.72 34.29 0)
+			(at 176.53 54.61 0)
 			(effects
 				(font
@@
 		)
 		(property "Value" "+5V"
-			(at 173.101 26.0858 0)
+			(at 176.911 46.4058 0)
 			(effects
 				(font
@@
 		)
 		(property "Footprint" ""
-			(at 172.72 30.48 0)
+			(at 176.53 50.8 0)
 			(effects
 				(font
@@
 		)
 		(property "Datasheet" ""
-			(at 172.72 30.48 0)
+			(at 176.53 50.8 0)
 			(effects
 				(font
@@
 		)
 		(property "Description" ""
-			(at 172.72 30.48 0)
+			(at 176.53 50.8 0)
 			(effects
 				(font

Commit message: I mixed up VSS and VDD
When connecting the LEDs in the schematic I flipped VSS (gnd) and VDD
(5v). The LED matrix won't work in the current wiring and needs to be
rerouted entirely.

Update routing for the first row.
Connections:
- net +5V: now also D100.3 (VDD), D101.3 (VDD), D102.3 (VDD), D103.3 (VDD), D104.3 (VDD), D105.3 (VDD), D106.3 (VDD), D107.3 (VDD), D108.3 (VDD), D109.3 (VDD), D110.3 (VDD), D111.3 (VDD), D112.3 (VDD), D113.3 (VDD), D114.3 (VDD), D115.3 (VDD), D116.3 (VDD), D117.3 (VDD), D118.3 (VDD), D119.3 (VDD), D120.3 (VDD), D121.3 (VDD), D122.3 (VDD), D123.3 (VDD), D124.3 (VDD), D125.3 (VDD), D126.3 (VDD), D127.3 (VDD), D128.3 (VDD), D129.3 (VDD), D130.3 (VDD), D131.3 (VDD), D132.3 (VDD), D133.3 (VDD), D134.3 (VDD), D135.3 (VDD), D136.3 (VDD), D137.3 (VDD), D138.3 (VDD), D139.3 (VDD), D140.3 (VDD), D141.3 (VDD), D142.3 (VDD), D143.3 (VDD), D144.3 (VDD), D145.3 (VDD), D146.3 (VDD), D147.3 (VDD), D148.3 (VDD), D149.3 (VDD), D150.3 (VDD), D151.3 (VDD), D152.3 (VDD), D153.3 (VDD), D154.3 (VDD), D155.3 (VDD), D156.3 (VDD), D157.3 (VDD), D158.3 (VDD), D159.3 (VDD), D160.3 (VDD), D161.3 (VDD), D162.3 (VDD), D163.3 (VDD), D164.3 (VDD), D83.3 (VDD), D84.3 (VDD), D85.3 (VDD), D86.3 (VDD), D87.3 (VDD), D88.3 (VDD), D89.3 (VDD), D90.3 (VDD), D91.3 (VDD), D92.3 (VDD), D93.3 (VDD), D94.3 (VDD), D95.3 (VDD), D96.3 (VDD), D97.3 (VDD), D98.3 (VDD), D99.3 (VDD); no longer D100.1 (VSS), D101.1 (VSS), D102.1 (VSS), D103.1 (VSS), D104.1 (VSS), D105.1 (VSS), D106.1 (VSS), D107.1 (VSS), D108.1 (VSS), D109.1 (VSS), D110.1 (VSS), D111.1 (VSS), D112.1 (VSS), D113.1 (VSS), D114.1 (VSS), D115.1 (VSS), D116.1 (VSS), D117.1 (VSS), D118.1 (VSS), D119.1 (VSS), D120.1 (VSS), D121.1 (VSS), D122.1 (VSS), D123.1 (VSS), D124.1 (VSS), D125.1 (VSS), D126.1 (VSS), D127.1 (VSS), D128.1 (VSS), D129.1 (VSS), D130.1 (VSS), D131.1 (VSS), D132.1 (VSS), D133.1 (VSS), D134.1 (VSS), D135.1 (VSS), D136.1 (VSS), D137.1 (VSS), D138.1 (VSS), D139.1 (VSS), D140.1 (VSS), D141.1 (VSS), D142.1 (VSS), D143.1 (VSS), D144.1 (VSS), D145.1 (VSS), D146.1 (VSS), D147.1 (VSS), D148.1 (VSS), D149.1 (VSS), D150.1 (VSS), D151.1 (VSS), D152.1 (VSS), D153.1 (VSS), D154.1 (VSS), D155.1 (VSS), D156.1 (VSS), D157.1 (VSS), D158.1 (VSS), D159.1 (VSS), D160.1 (VSS), D161.1 (VSS), D162.1 (VSS), D163.1 (VSS), D164.1 (VSS), D83.1 (VSS), D84.1 (VSS), D85.1 (VSS), D86.1 (VSS), D87.1 (VSS), D88.1 (VSS), D89.1 (VSS), D90.1 (VSS), D91.1 (VSS), D92.1 (VSS), D93.1 (VSS), D94.1 (VSS), D95.1 (VSS), D96.1 (VSS), D97.1 (VSS), D98.1 (VSS), D99.1 (VSS)
- net GND: now also D100.1 (VSS), D101.1 (VSS), D102.1 (VSS), D103.1 (VSS), D104.1 (VSS), D105.1 (VSS), D106.1 (VSS), D107.1 (VSS), D108.1 (VSS), D109.1 (VSS), D110.1 (VSS), D111.1 (VSS), D112.1 (VSS), D113.1 (VSS), D114.1 (VSS), D115.1 (VSS), D116.1 (VSS), D117.1 (VSS), D118.1 (VSS), D119.1 (VSS), D120.1 (VSS), D121.1 (VSS), D122.1 (VSS), D123.1 (VSS), D124.1 (VSS), D125.1 (VSS), D126.1 (VSS), D127.1 (VSS), D128.1 (VSS), D129.1 (VSS), D130.1 (VSS), D131.1 (VSS), D132.1 (VSS), D133.1 (VSS), D134.1 (VSS), D135.1 (VSS), D136.1 (VSS), D137.1 (VSS), D138.1 (VSS), D139.1 (VSS), D140.1 (VSS), D141.1 (VSS), D142.1 (VSS), D143.1 (VSS), D144.1 (VSS), D145.1 (VSS), D146.1 (VSS), D147.1 (VSS), D148.1 (VSS), D149.1 (VSS), D150.1 (VSS), D151.1 (VSS), D152.1 (VSS), D153.1 (VSS), D154.1 (VSS), D155.1 (VSS), D156.1 (VSS), D157.1 (VSS), D158.1 (VSS), D159.1 (VSS), D160.1 (VSS), D161.1 (VSS), D162.1 (VSS), D163.1 (VSS), D164.1 (VSS), D83.1 (VSS), D84.1 (VSS), D85.1 (VSS), D86.1 (VSS), D87.1 (VSS), D88.1 (VSS), D89.1 (VSS), D90.1 (VSS), D91.1 (VSS), D92.1 (VSS), D93.1 (VSS), D94.1 (VSS), D95.1 (VSS), D96.1 (VSS), D97.1 (VSS), D98.1 (VSS), D99.1 (VSS); no longer D100.3 (VDD), D101.3 (VDD), D102.3 (VDD), D103.3 (VDD), D104.3 (VDD), D105.3 (VDD), D106.3 (VDD), D107.3 (VDD), D108.3 (VDD), D109.3 (VDD), D110.3 (VDD), D111.3 (VDD), D112.3 (VDD), D113.3 (VDD), D114.3 (VDD), D115.3 (VDD), D116.3 (VDD), D117.3 (VDD), D118.3 (VDD), D119.3 (VDD), D120.3 (VDD), D121.3 (VDD), D122.3 (VDD), D123.3 (VDD), D124.3 (VDD), D125.3 (VDD), D126.3 (VDD), D127.3 (VDD), D128.3 (VDD), D129.3 (VDD), D130.3 (VDD), D131.3 (VDD), D132.3 (VDD), D133.3 (VDD), D134.3 (VDD), D135.3 (VDD), D136.3 (VDD), D137.3 (VDD), D138.3 (VDD), D139.3 (VDD), D140.3 (VDD), D141.3 (VDD), D142.3 (VDD), D143.3 (VDD), D144.3 (VDD), D145.3 (VDD), D146.3 (VDD), D147.3 (VDD), D148.3 (VDD), D149.3 (VDD), D150.3 (VDD), D151.3 (VDD), D152.3 (VDD), D153.3 (VDD), D154.3 (VDD), D155.3 (VDD), D156.3 (VDD), D157.3 (VDD), D158.3 (VDD), D159.3 (VDD), D160.3 (VDD), D161.3 (VDD), D162.3 (VDD), D163.3 (VDD), D164.3 (VDD), D83.3 (VDD), D84.3 (VDD), D85.3 (VDD), D86.3 (VDD), D87.3 (VDD), D88.3 (VDD), D89.3 (VDD), D90.3 (VDD), D91.3 (VDD), D92.3 (VDD), D93.3 (VDD), D94.3 (VDD), D95.3 (VDD), D96.3 (VDD), D97.3 (VDD), D98.3 (VDD), D99.3 (VDD)

Commit message: Use a bigger fuse
500mA was popping when all the LEDs were connected at default
brightness. This took a long time to figure out sadly.
Parts:
- FU2: value 500mA -> 750mA
Changed lines of the file:
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@@
 			)
 		)
-		(property "Value" "500mA"
+		(property "Value" "750mA"
 			(at 166.37 47.9044 90)
 			(effects

Commit message: Add first draft of lcsc part numbers
Need to double check these one more time.
Parts:
- C1, C2: LCSC Part # (none) -> C105623
- C3: LCSC Part # (none) -> C472813
- C4, C5, C6: LCSC Part # (none) -> C62912
- C7: LCSC Part # (none) -> C307520
- D1, D10, D11, D12, D13, D14, D15, D16, D165, D17, D18, D19, D2, D20, D21, D22, D23, D24, D25, D26, D27, D28, D29, D3, D30, D31, D32, D33, D34, D35, D36, D37, D38, D39, D4, D40, D41, D42, D43, D44, D45, D46, D47, D48, D49, D5, D50, D51, D52, D53, D54, D55, D56, D57, D58, D59, D6, D60, D61, D62, D63, D64, D65, D66, D67, D68, D69, D7, D70, D71, D72, D73, D74, D75, D76, D77, D78, D79, D8, D80, D81, D82, D9: LCSC Part # (none) -> C7420318
- D100, D101, D102, D103, D104, D105, D106, D107, D108, D109, D110, D111, D112, D113, D114, D115, D116, D117, D118, D119, D120, D121, D122, D123, D124, D125, D126, D127, D128, D129, D130, D131, D132, D133, D134, D135, D136, D137, D138, D139, D140, D141, D142, D143, D144, D145, D146, D147, D148, D149, D150, D151, D152, D153, D154, D155, D156, D157, D158, D159, D160, D161, D162, D163, D164, D83, D84, D85, D86, D87, D88, D89, D90, D91, D92, D93, D94, D95, D96, D97, D98, D99: LCSC Part # (none) -> C5149201
- F10: now not fitted
- FU2: LCSC Part # (none) -> C5144563
- J2: LCSC Part # (none) -> C696092
- R1, R8: LCSC Part # (none) -> C180849
- R6, R7: LCSC Part # (none) -> C413152
- SW1: LCSC Part # (none) -> C720467
- SW2: LCSC Part # (none) -> C470748
- U1: LCSC Part # (none) -> C44854
- Y1: LCSC Part # (none) -> C258944

Commit message: Fix part numbers
Parts:
- C4, C5, C6: LCSC Part # C62912 -> C49678
- F10: now fitted
Changed lines of the file:
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@@
 			)
 		)
-		(property "LCSC Part #" "C62912"
+		(property "LCSC Part #" "C49678"
 			(at 21.59 118.11 0)
 			(effects
@@
 			)
 		)
-		(property "LCSC Part #" "C62912"
+		(property "LCSC Part #" "C49678"
 			(at 33.02 118.11 0)
 			(effects
@@
 			)
 		)
-		(property "LCSC Part #" "C62912"
+		(property "LCSC Part #" "C49678"
 			(at 43.18 118.11 0)
 			(effects
@@
 		(in_bom yes)
 		(on_board yes)
-		(dnp yes)
+		(dnp no)
 		(property "Reference" "F10"
 			(at 347.5482 29.8958 0)
